File: hardware/powiloc.sch (KiCad schematic (older format))
At the start: 32 parts

Commit message: Update schematic design
Parts:
- added D3: LED_PWR, LED_THT:LED_D5.0mm, symbol Device:LED_Small
- added D4: LED_STAT, LED_THT:LED_D5.0mm, symbol Device:LED_Small
- added J10: BAT-, Connector_PinHeader_2.54mm:PinHeader_1x01_P2.54mm_Vertical, symbol Connector_Generic:Conn_01x01
- added J6: periph_conn_1, Connector_PinHeader_2.54mm:PinHeader_2x03_P2.54mm_Vertical, symbol Connector_Generic:Conn_02x03_Odd_Even
- added J9: BAT+, Connector_PinHeader_2.54mm:PinHeader_1x01_P2.54mm_Vertical, symbol Connector_Generic:Conn_01x01
- added R10, R7, R9: 4k7, Resistor_THT:R_Axial_DIN0207_L6.3mm_D2.5mm_P7.62mm_Horizontal, symbol Device:R_Small
- added R11, R12: 1k, Resistor_THT:R_Axial_DIN0207_L6.3mm_D2.5mm_P7.62mm_Horizontal, symbol Device:R_Small
- added SW3: SW_LED_PWR, Connector_PinHeader_2.54mm:PinHeader_1x02_P2.54mm_Vertical, symbol Switch:SW_SPST
- C1, C2, C3: renamed from C?; footprint (none) -> Capacitor_THT:C_Disc_D5.0mm_W2.5mm_P5.00mm
- C4, C5: renamed from C?; value 22p -> 20p; footprint (none) -> Capacitor_THT:C_Disc_D5.0mm_W2.5mm_P2.50mm
- C6, C7: renamed from C?; footprint (none) -> Capacitor_THT:C_Disc_D5.0mm_W2.5mm_P2.50mm
- D1, D2: renamed from D?; footprint (none) -> Diode_THT:D_DO-41_SOD81_P7.62mm_Horizontal
- J1: renamed from J?; value SW_PWR -> SW_PWR_BAT; footprint (none) -> Connector_PinHeader_2.54mm:PinHeader_1x02_P2.54mm_Vertical
- J2, J3: renamed from J?; footprint (none) -> Connector_PinHeader_2.54mm:PinHeader_2x03_P2.54mm_Vertical
- J4, J5: renamed from J?; footprint (none) -> Connector_PinHeader_2.54mm:PinHeader_1x04_P2.54mm_Vertical
- J8: renamed from J?; footprint (none) -> Connector_Coaxial:SMA_Amphenol_132134-16_Vertical
- R1, R2, R3, R4, R5, R6, R8: renamed from R?; footprint (none) -> Resistor_THT:R_Axial_DIN0207_L6.3mm_D2.5mm_P7.62mm_Horizontal
- SW1: renamed from SW?; value SW_SPST -> SW_TRIG; footprint (none) -> Button_Switch_THT:SW_PUSH_6mm
- SW2: renamed from SW?; footprint (none) -> Button_Switch_THT:SW_PUSH_6mm
- U3: renamed from U?; footprint (none) -> RF_Module:HOPERF_RFM9XW_SMD
- Y1: renamed from Y?; value 16MHz -> 12MHz; footprint (none) -> Crystal:Crystal_HC49-U_Vertical
- gave numbers to parts that had none: 6
Connections:
- net VCC is gone; now on net 3.3V: R8.1
- net 3.3V: now also J6.1 (Pin_1), R10.1, R7.1, R9.1, SW3.1 (A)
- net 3.3V_SW: now also J6.5 (Pin_5)
- net BAT+: now also J9.1 (Pin_1)
- net GND: now also J10.1 (Pin_1), J6.3 (Pin_3), R11.1, R12.1
- net I2C_SCL: now also J6.6 (Pin_6), R10.2
- net I2C_SDA: now also J6.4 (Pin_4), R9.2
- net PWR_SW: now also U4.24 (PC1); no longer U4.25 (PC2)
- net RADIO_DIO5: now also U5.25 (PC2); no longer U5.26 (PC3)
- net TRIG_BTN: now also U4.25 (PC2); no longer U4.26 (PC3)
- net VBUS: now also J2.2 (Pin_2), J3.2 (Pin_2)
- net SW_LED_STAT: now reaches U4.13 (PD7)
- net SW_LED_STAT: now also D4.2 (A)
- new net: D3.1 (K), R11.2
- new net: D3.2 (A), SW3.2 (B)
- new net: D4.1 (K), R12.2
- new net I2C_SMBALERT: J6.2 (Pin_2), R7.2, U4.26 (PC3), U5.26 (PC3)
- no-connect marks 0 -> 21
Other:
- note added: "Battery Connector"
- note added: "I2C Bus"
- note added: "LEDs*"
- note added: "Peripheral\nConnectors*"
- note added: "Trigger button"
- note removed: "Trigger\nbutton"
- moved on the sheet: C1, C2, C3, C4, C5, D1, D2, J1, J2, J3, J4, J5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

Commit message: PCB Placement
Parts:
- removed J10: BAT-, Connector_PinHeader_2.54mm:PinHeader_1x01_P2.54mm_Vertical, symbol Connector_Generic:Conn_01x01
- removed J3: 328p_radio_ISP, Connector_PinHeader_2.54mm:PinHeader_2x03_P2.54mm_Vertical, symbol Connector_Generic:Conn_02x03_Odd_Even
- removed J9: BAT+, Connector_PinHeader_2.54mm:PinHeader_1x01_P2.54mm_Vertical, symbol Connector_Generic:Conn_01x01
- added J3: SW_ISP_MCU, Connector_PinHeader_2.54mm:PinHeader_1x03_P2.54mm_Vertical, symbol Connector_Generic:Conn_01x03
- added J7: BATT, Connector_JST:JST_XH_B2B-XH-A_1x02_P2.50mm_Vertical, symbol Connector_Generic:Conn_01x02
- added J9: MCU_TX, Connector_PinSocket_2.54mm:PinSocket_1x03_P2.54mm_Vertical, symbol Connector_Generic:Conn_01x03
- added R13: 10k, Resistor_THT:R_Axial_DIN0207_L6.3mm_D2.5mm_P7.62mm_Horizontal, symbol Device:R_Small
- added SW4: SW_LED_STAT, Connector_PinHeader_2.54mm:PinHeader_1x02_P2.54mm_Vertical, symbol Switch:SW_SPST
- added SW5: SW_RADIO_RST, Button_Switch_THT:SW_PUSH_6mm, symbol Switch:SW_SPST
- J2: value 328p_main_ISP -> MCU_ISP
- J4, J5: footprint Connector_PinHeader_2.54mm:PinHeader_1x04_P2.54mm_Vertical -> Connector_PinSocket_2.54mm:PinSocket_1x04_P2.54mm_Vertical
- J8: footprint Connector_Coaxial:SMA_Amphenol_132134-16_Vertical -> Connector_Coaxial:SMA_Amphenol_132289_EdgeMount
- Q1, Q2: footprint Package_TO_SOT_THT:TO-220-3_Vertical -> Package_TO_SOT_THT:TO-220-3_Horizontal_TabDown
- SW2: value SW_RST -> SW_MAIN_RST
- U2: footprint (none) -> powiloc-custom:USBPCB
- U4, U5: footprint Package_DIP:DIP-28_W7.62mm -> Package_DIP:DIP-28_W7.62mm_Socket
Connections:
- net RADIO_MISO is gone; now on net SPI_MISO: U3.2 (MISO), U5.18 (PB4)
- net RADIO_MOSI is gone; now on net SPI_MOSI: U3.3 (MOSI), U5.17 (PB3)
- net RADIO_SCK is gone; now on net SPI_SCK: U3.4 (SCK), U5.19 (PB5)
- net 3.3V: now also R13.1
- net BAT+: now also J7.2 (Pin_2)
- net GND: now also J7.1 (Pin_1), J9.2 (Pin_2), SW5.1 (A)
- net SW_LED_STAT: now also SW4.1 (A); no longer D4.2 (A)
- net RADIO_TX: now reaches U5.3 (PD1)
- net RADIO_TX: now also J9.1 (Pin_1)
- net GPS_RX renamed MAIN_TX
- net MAIN_TX: now also J9.3 (Pin_3)
- net GPS_TX renamed MAIN_RX
- net MAIN_MISO renamed SPI_MISO
- net MAIN_MOSI renamed SPI_MOSI
- net MAIN_SCK renamed SPI_SCK
- net NRST renamed NRST_MAIN_MCU
- net NRST_MAIN_MCU: now also J3.1 (Pin_1); no longer J2.5 (Pin_5), U5.1 (~RESET~/PC6)
- new net: J2.5 (Pin_5), J3.2 (Pin_2)
- new net: D4.2 (A), SW4.2 (B)
- new net NRST_RADIO_MCU: J3.3 (Pin_3), R13.2, SW5.2 (B), U5.1 (~RESET~/PC6)
- no-connect marks 21 -> 20
Other:
- note added: "MCU UART TX"
- note added: "Radio Reset button"
- moved on the sheet: R6, SW1

Commit message: Corrupt save
Parts:
- removed J1: SW_PWR_BAT, Connector_PinHeader_2.54mm:PinHeader_1x02_P2.54mm_Vertical, symbol Connector_Generic:Conn_01x02
- added J1: periph_conn_2, Connector_PinHeader_2.54mm:PinHeader_2x03_P2.54mm_Vertical, symbol Connector_Generic:Conn_02x03_Odd_Even
- added T1, T2, T5: taper, powiloc-custom:uwT0.50_0.40_1.00_1.46_1.20, symbol powiloc-custom:taper
- added T3, T4: taper, powiloc-custom:uwT0.50_0.15_1.00_1.24_3.00, symbol powiloc-custom:taper
Connections:
- net 3.3V: now also J1.1 (Pin_1)
- net 3.3V_SW: now also J1.5 (Pin_5)
- net BAT+: now also Q1.3 (S)
- net GND: now also J1.3 (Pin_3), T2.1
- net I2C_SCL: now also J1.6 (Pin_6)
- net I2C_SDA: now also J1.4 (Pin_4)
- net I2C_SMBALERT: now also J1.2 (Pin_2)
- net USB_D+: now also U4.5 (PD3); no longer U4.4 (PD2)
- net USB_D-: now also U4.4 (PD2); no longer U4.5 (PD3)
- net VBUS: now also T1.1
- net at J8.1 (In), U3.9 (ANT): now also T5.1
- net at R3.1, R4.1, U2.2 (D-): now also T4.1
- net at R5.1, U2.3 (D+): now also T3.1
Other:
- moved on the sheet: R4, R5
Changed lines of the file:
@@
 	1    0    0    -1
 $EndComp
+Text GLabel 2400 6700 2    50   Input ~ 0
+USB_D+
 Text GLabel 2400 6600 2    50   Input ~ 0
+USB_D-
+Text GLabel 8300 1450 0    50   Input ~ 0
 USB_D+
-Text GLabel 2400 6700 2    50   Input ~ 0
-USB_D-
-Text GLabel 8350 1450 0    50   Input ~ 0
-USB_D+
-Text GLabel 8350 1350 0    50   Input ~ 0
+Text GLabel 8300 1350 0    50   Input ~ 0
 USB_D-
 Wire Wire Line
@@
 L Device:R_Small R5
 U 1 1 60106E17
-P 8500 1450
-F 0 "R5" V 8400 1400 50  0000 C CNN
-F 1 "68" V 8400 1550 50  0000 C CNN
-F 2 "Resistor_THT:R_Axial_DIN0207_L6.3mm_D2.5mm_P7.62mm_Horizontal" H 8500 1450 50  0001 C CNN
-F 3 "~" H 8500 1450 50  0001 C CNN
-	1    8500 1450
+P 8450 1450
+F 0 "R5" V 8350 1400 50  0000 C CNN
+F 1 "68" V 8350 1550 50  0000 C CNN
+F 2 "Resistor_THT:R_Axial_DIN0207_L6.3mm_D2.5mm_P7.62mm_Horizontal" H 8450 1450 50  0001 C CNN
+F 3 "~" H 8450 1450 50  0001 C CNN
+	1    8450 1450
 	0    1    -1   0
 $EndComp
@@
 L Device:R_Small R4
 U 1 1 6012B34F
-P 8500 1350
-F 0 "R4" V 8400 1300 50  0000 C CNN
-F 1 "68" V 8400 1450 50  0000 C CNN
-F 2 "Resistor_THT:R_Axial_DIN0207_L6.3mm_D2.5mm_P7.62mm_Horizontal" H 8500 1350 50  0001 C CNN
-F 3 "~" H 8500 1350 50  0001 C CNN
-	1    8500 1350
+P 8450 1350
+F 0 "R4" V 8350 1300 50  0000 C CNN
+F 1 "68" V 8350 1450 50  0000 C CNN
+F 2 "Resistor_THT:R_Axial_DIN0207_L6.3mm_D2.5mm_P7.62mm_Horizontal" H 8450 1350 50  0001 C CNN
+F 3 "~" H 8450 1350 50  0001 C CNN
+	1    8450 1350
 	0    1    1    0
 $EndComp
 Wire Wire Line
-	8400 1350 8350 1350
-Wire Wire Line
-	8350 1450 8400 1450
+	8350 1350 8300 1350
+Wire Wire Line
+	8300 1450 8350 1450
 Wire Wire Line
 	8900 1250 8900 1200
@@
 	8750 850  8750 900
 Wire Wire Line
-	7800 1200 8900 1200
+	7800 1200 8400 1200
 Wire Notes Line
 	7500 2000 9550 2000
@@
 Wire Wire Line
 	8750 1100 8750 1350
-Wire Wire Line
-	8600 1350 8750 1350
-Connection ~ 8750 1350
-Wire Wire Line
-	8750 1350 8950 1350
-Wire Wire Line
-	8600 1450 8950 1450
 $Comp
 L Device:C_Small C6
@@
 RADIO_DIO5
 Wire Wire Line
-	7750 5000 8150 5000
+	7750 5000 7850 5000
 Text GLabel 4800 5800 2    50   Input ~ 0
 RADIO_DIO5
@@
 Wire Notes Line
 	4900 1750 6000 1750
-$Comp
-L Connector_Generic:Conn_01x02 J1
-U 1 1 60157CEE
-P 1050 1000
-F 0 "J1" V 1100 1100 50  0000 L BNN
-F 1 "SW_PWR_BAT" V 1000 1050 50  0000 L CNN
-F 2 "Connector_PinHeader_2.54mm:PinHeader_1x02_P2.54mm_Vertical" H 1050 1000 50  0001 C CNN
-F 3 "~" H 1050 1000 50  0001 C CNN
-	1    1050 1000
-	0    -1   -1   0
-$EndComp
-Wire Wire Line
-	1150 1200 1500 1200
 $Comp
 L Device:C_Small C1
@@
 	9450 2050 11150 2050
 Wire Notes Line
-	11150 3000 9450 3000
+	11150 3450 9450 3450
 NoConn ~ 7750 5300
 NoConn ~ 7750 5400
@@
 $EndComp
 Wire Wire Line
-	850  1200 1050 1200
-Wire Wire Line
 	1000 2950 1050 2950
 Connection ~ 1000 2950
@@
 Wire Wire Line
 	8950 1550 8900 1550
-Wire Wire Line
-	8900 1550 8900 1600
-Wire Wire Line
-	8900 1600 7800 1600
 Connection ~ 7800 1600
 Wire Wire Line
@@
 	1000 3150 1050 3150
 Connection ~ 1000 3150
-Wire Notes Line
-	9450 2050 9450 3000
-Wire Notes Line
-	11150 3000 11150 2050
 $Comp
 L Switch:SW_SPST SW4
@@
 Wire Notes Line
 	4900 3350 4900 2700
+Wire Wire Line
+	850  1200 1500 1200
+$Comp
+L Connector_Generic:Conn_02x03_Odd_Even J1
+U 1 1 605D268F
+P 10200 3150
+F 0 "J1" H 10250 3467 50  0000 C CNN
+F 1 "periph_conn_2" H 10250 3376 50  0000 C CNN
+F 2 "Connector_PinHeader_2.54mm:PinHeader_2x03_P2.54mm_Vertical" H 10200 3150 50  0001 C CNN
+F 3 "~" H 10200 3150 50  0001 C CNN
+	1    10200 3150
+	1    0    0    -1
+$EndComp
+Text GLabel 10000 3050 0    50   Input ~ 0
+3.3V
+$Comp
+L power:GND #PWR09
+U 1 1 605D2C8C
+P 9550 3200
+F 0 "#PWR09" H 9550 2950 50  0001 C CNN
+F 1 "GND" H 9555 3027 50  0000 C CNN
+F 2 "" H 9550 3200 50  0001 C CNN
+F 3 "" H 9550 3200 50  0001 C CNN
+	1    9550 3200
+	1    0    0    -1
+$EndComp
+Text GLabel 10500 3250 2    50   Input ~ 0
+I2C_SCL
+Text GLabel 10500 3150 2    50   Input ~ 0
+I2C_SDA
+Text GLabel 10500 3050 2    50   Input ~ 0
+I2C_SMBALERT
+Text GLabel 10000 3250 0    50   Input ~ 0
+3.3V_SW
+Wire Wire Line
+	9550 3150 10000 3150
+Wire Wire Line
+	9550 3200 9550 3150
+Wire Notes Line
+	9450 2050 9450 3450
+Wire Notes Line
+	11150 2050 11150 3450
+$Comp
+L pollex-logo:LOGO #G1
+U 1 1 606E97B4
+P 10450 6900
+F 0 "#G1" H 10450 6780 60  0001 C CNN
+F 1 "LOGO" H 10450 7020 60  0001 C CNN
+F 2 "" H 10450 6900 50  0001 C CNN
+F 3 "" H 10450 6900 50  0001 C CNN
+	1    10450 6900
+	1    0    0    -1
+$EndComp
+$Comp
+L Graphic:Logo_Open_Hardware_Small #LOGO1
+U 1 1 606ECD78
+P 9200 6900
+F 0 "#LOGO1" H 9200 7175 50  0001 C CNN
+F 1 "Logo_Open_Hardware_Small" H 9200 6675 50  0001 C CNN
+F 2 "" H 9200 6900 50  0001 C CNN
+F 3 "~" H 9200 6900 50  0001 C CNN
+	1    9200 6900
+	1    0    0    -1
+$EndComp
+$Comp
+L powiloc-custom:taper T5
+U 1 1 6077932E
+P 7850 4900
+F 0 "T5" H 7950 5050 50  0001 C CNN
+F 1 "taper" H 7800 5050 50  0000 L CNN
+F 2 "powiloc-custom:uwT0.50_0.40_1.00_1.46_1.20" H 8000 5000 50  0001 C CNN
+F 3 "" H 7900 4850 50  0001 C CNN
+	1    7850 4900
+	1    0    0    -1
+$EndComp
+Wire Wire Line
+	7850 4900 7850 5000
+Connection ~ 7850 5000
+Wire Wire Line
+	7850 5000 8150 5000
+$Comp
+L powiloc-custom:taper T4
+U 1 1 60782203
+P 8850 1700
+F 0 "T4" H 8950 1850 50  0001 C CNN
+F 1 "taper" H 8800 1850 50  0000 L CNN
+F 2 "powiloc-custom:uwT0.50_0.15_1.00_1.24_3.00" H 9000 1800 50  0001 C CNN
+F 3 "" H 8900 1650 50  0001 C CNN
+	1    8850 1700
+	-1   0    0    1
+$EndComp
+$Comp
+L powiloc-custom:taper T2
+U 1 1 60791D80
+P 8250 1700
+F 0 "T2" H 8350 1850 50  0001 C CNN
+F 1 "taper" H 8200 1850 50  0000 L CNN
+F 2 "powiloc-custom:uwT0.50_0.40_1.00_1.46_1.20" H 8400 1800 50  0001 C CNN
+F 3 "" H 8300 1650 50  0001 C CNN
+	1    8250 1700
+	-1   0    0    1
+$EndComp
+$Comp
+L powiloc-custom:taper T1
+U 1 1 60791FFC
+P 8400 1100
+F 0 "T1" H 8500 1250 50  0001 C CNN
+F 1 "taper" H 8350 1250 50  0000 L CNN
+F 2 "powiloc-custom:uwT0.50_0.40_1.00_1.46_1.20" H 8550 1200 50  0001 C CNN
+F 3 "" H 8450 1050 50  0001 C CNN
+	1    8400 1100
+	1    0    0    -1
+$EndComp
+Wire Wire Line
+	8400 1100 8400 1200
+Connection ~ 8400 1200
+Wire Wire Line
+	8400 1200 8900 1200
+Wire Wire Line
+	7800 1600 8250 1600
+Wire Wire Line
+	8250 1700 8250 1600
+Wire Wire Line
+	8550 1700 8550 1450
+Connection ~ 8550 1450
+Wire Wire Line
+	8750 1350 8850 1350
+Wire Wire Line
+	8900 1550 8900 1600
+Connection ~ 8250 1600
+Wire Wire Line
+	8250 1600 8900 1600
+Wire Wire Line
+	8550 1350 8750 1350
+Connection ~ 8750 1350
+$Comp
+L powiloc-custom:taper T3
+U 1 1 60783E09
+P 8550 1700
+F 0 "T3" H 8650 1850 50  0001 C CNN
+F 1 "taper" H 8500 1850 50  0000 L CNN
+F 2 "powiloc-custom:uwT0.50_0.15_1.00_1.24_3.00" H 8700 1800 50  0001 C CNN
+F 3 "" H 8600 1650 50  0001 C CNN
+	1    8550 1700
+	-1   0    0    1
+$EndComp
+Wire Wire Line
+	8550 1450 8950 1450
+Wire Wire Line
+	8850 1700 8850 1350
+Connection ~ 8850 1350
+Wire Wire Line
+	8850 1350 8950 1350
 $EndSCHEMATC
