File: hardware/powiloc.kicad_pcb (KiCad board)
At the start: 2 copper layers, 42 parts, among them J1 SW_PWR_BAT, J10 BAT-, J2 328p_main_ISP, J3 328p_radio_ISP, J4 neo_gps_conn, J5 oled_conn, J6 periph_conn_1, J8 radio_ant_conn**, J9 BAT+, Q1 IRF740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

Commit message: PCB Placement
Parts:
- removed J10: BAT-, Connector_PinHeader_2.54mm:PinHeader_1x01_P2.54mm_Vertical
- added J7: BATT, Connector_JST:JST_XH_B2B-XH-A_1x02_P2.50mm_Vertical, F.Cu at (122.2, 134.4)
- added R13: 10k, Resistor_THT:R_Axial_DIN0207_L6.3mm_D2.5mm_P7.62mm_Horizontal, F.Cu at (159.5, 113.8)
- added SW4: SW_LED_STAT, Connector_PinHeader_2.54mm:PinHeader_1x02_P2.54mm_Vertical, F.Cu at (129.8, 70.6)
- added SW5: SW_RADIO_RST, Button_Switch_THT:SW_PUSH_6mm, F.Cu at (160.0, 105.7)
- added U2: USB Conn, powiloc-custom:USBPCB, F.Cu at (142.2, 152.3)
- J2: value 328p_main_ISP -> MCU_ISP
- J3: value 328p_radio_ISP -> SW_ISP_MCU; footprint Connector_PinHeader_2.54mm:PinHeader_2x03_P2.54mm_Vertical -> Connector_PinHeader_2.54mm:PinHeader_1x03_P2.54mm_Vertical
- J4, J5: footprint Connector_PinHeader_2.54mm:PinHeader_1x04_P2.54mm_Vertical -> Connector_PinSocket_2.54mm:PinSocket_1x04_P2.54mm_Vertical
- J8: footprint Connector_Coaxial:SMA_Amphenol_132134-16_Vertical -> Connector_Coaxial:SMA_Amphenol_132289_EdgeMount
- J9: value BAT+ -> MCU_TX; footprint Connector_PinHeader_2.54mm:PinHeader_1x01_P2.54mm_Vertical -> Connector_PinSocket_2.54mm:PinSocket_1x03_P2.54mm_Vertical
- Q1, Q2: footprint Package_TO_SOT_THT:TO-220-3_Vertical -> Package_TO_SOT_THT:TO-220-3_Horizontal_TabDown
- R11, R12: value 500 -> 1k
- SW2: value SW_RST -> SW_MAIN_RST
- U4, U5: footprint Package_DIP:DIP-28_W7.62mm -> Package_DIP:DIP-28_W7.62mm_Socket
- moved J1 262.2 mm to (131.3, 135.4), turned to 270 degrees
- moved C3 258.2 mm to (137.7, 137.7)
- moved C6 251.2 mm to (124.7, 102.6), turned to 90 degrees
- moved R6 247.6 mm to (138.0, 123.4)
- moved U1 243.0 mm to (128.8, 131.1)
- moved SW3 242.7 mm to (122.4, 70.6), turned to 270 degrees
- moved D4 236.5 mm to (129.8, 65.0), turned to 180 degrees
- moved D3 234.1 mm to (122.4, 65.0), turned to 180 degrees
- moved R4 232.9 mm to (145.4, 134.9), turned to 90 degrees
- moved J9 231.7 mm to (166.4, 128.5), turned to 180 degrees
- moved R11 230.3 mm to (128.3, 81.5), turned to 90 degrees
- moved R7 228.1 mm to (149.0, 131.2), turned to 90 degrees
- moved D1 227.8 mm to (136.0, 127.0), turned to 270 degrees
- moved R10 226.7 mm to (155.1, 131.2), turned to 90 degrees
- moved C2 226.3 mm to (127.5, 123.7)
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Connections:
- net GPS_TX renamed MAIN_RX
- D4 pad 2: SW_LED_STAT -> Net-(D4-Pad2)
- J2 pad 1: MAIN_MISO -> SPI_MISO
- J2 pad 3: MAIN_SCK -> SPI_SCK
- J2 pad 4: MAIN_MOSI -> SPI_MOSI
- J2 pad 5: NRST -> Net-(J2-Pad5)
- J3 pad 1: RADIO_MISO -> NRST_MAIN_MCU
- J3 pad 2: VBUS -> Net-(J2-Pad5)
- J3 pad 3: RADIO_SCK -> NRST_RADIO_MCU
- J4 pad 2: GPS_RX -> MAIN_TX
- J9 pad 1: BAT+ -> RADIO_TX
- R8 pad 2: NRST -> NRST_MAIN_MCU
- SW2 pad 2: NRST -> NRST_MAIN_MCU
- U3 pad 2: RADIO_MISO -> SPI_MISO
- U3 pad 3: RADIO_MOSI -> SPI_MOSI
- U3 pad 4: RADIO_SCK -> SPI_SCK
- U4 pad 1: NRST -> NRST_MAIN_MCU
- U4 pad 17: MAIN_MOSI -> SPI_MOSI
- U4 pad 18: MAIN_MISO -> SPI_MISO
- U4 pad 19: MAIN_SCK -> SPI_SCK
- U4 pad 3: GPS_RX -> MAIN_TX
- U5 pad 1: NRST -> NRST_RADIO_MCU
- U5 pad 17: RADIO_MOSI -> SPI_MOSI
- U5 pad 18: RADIO_MISO -> SPI_MISO
- U5 pad 19: RADIO_SCK -> SPI_SCK
- U5 pad 3: Net-(U5-Pad3) -> RADIO_TX
Other:
- board outline added: 55.9 x 92.7 mm
- board text added: "+"
- board text added: "++"
- board text added: "-"
- board text added: "ANT"
- board text added: "BAT_CONN"
- board text added: "DATA+"
- board text added: "DATA-"
- board text added: "DISPLAY"
- board text added: "GND"
- board text added: "GPS"
- board text added: "ISP"
- board text added: "LORA_RADIO"
- board text added: "MAIN"
- board text added: "MAIN_MCU"
- board text added: "PERIPHERAL"
- board text added: "PWR"
- board text added: "RADIO"
- board text added: "RADIO_MCU"
- board text added: "RST MAIN"
- board text added: "RST RADIO"
- board text added: "SCL"
- board text added: "SDA"
- board text added: "SMBALERT"
- board text added: "STATUS"
- board text added: "SW_BAT"
- board text added: "UART"
- board text added: "VBUS"

Commit message: Corrupt save
Parts:
- added T1: taper, powiloc-custom:uwT0.50_0.40_1.00_1.46_1.20, F.Cu at (146.1, 137.9)
- added T2: taper, powiloc-custom:uwT0.50_0.40_1.00_1.46_1.20, F.Cu at (138.4, 137.8)
- added T3: taper, powiloc-custom:uwT0.50_0.15_1.00_1.24_3.00, F.Cu at (141.2, 136.1)
- added T4: taper, powiloc-custom:uwT0.50_0.15_1.00_1.24_3.00, F.Cu at (143.3, 136.1)
- added T5: taper, powiloc-custom:uwT0.50_0.40_1.00_1.46_1.20, F.Cu at (124.7, 60.5)
- J1: value SW_PWR_BAT -> periph_conn_2; footprint Connector_PinHeader_2.54mm:PinHeader_1x02_P2.54mm_Vertical -> Connector_PinHeader_2.54mm:PinHeader_2x03_P2.54mm_Vertical
- moved J1 48.5 mm to (119.1, 88.4), turned to 0 degrees
- moved J6 47.4 mm to (119.1, 79.2), turned to 0 degrees
- moved R2 45.1 mm to (167.5, 109.7)
- moved Q2 45.1 mm to (161.0, 106.8)
- moved J2 44.9 mm to (121.6, 70.0)
- moved SW2 37.1 mm to (166.4, 134.6), turned to 180 degrees
- moved D3 37.0 mm to (159.0, 59.3)
- moved D4 37.0 mm to (166.4, 59.3)
- moved SW3 37.0 mm to (159.0, 64.9)
- moved SW4 34.4 mm to (163.7, 64.9), turned to 90 degrees
- moved J8 34.0 mm to (124.7, 56.9)
- moved R11 32.1 mm to (157.7, 68.7), turned to 0 degrees
- moved J3 30.8 mm to (129.2, 65.0), turned to 0 degrees
- moved SW5 29.4 mm to (154.9, 134.6), turned to 180 degrees
- moved R12 28.2 mm to (157.7, 71.8), turned to 0 degrees
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Connections:
- J1 pad 1: BAT+ -> 3.3V
- J1 pad 2: Net-(J1-Pad2) -> I2C_SMBALERT
- Q1 pad 3: Net-(J1-Pad2) -> BAT+
- U4 pad 4: USB_D+ -> USB_D-
- U4 pad 5: USB_D- -> USB_D+
Routing:
- net 3.3V_SW: track 0.00 -> 118.4 mm, vias 0 -> 3
- net I2C_SCL: track 0.00 -> 114.7 mm, vias 0 -> 3
- net I2C_SDA: track 0.00 -> 109.2 mm, vias 0 -> 3
- net NRST_MAIN_MCU: track 0.00 -> 104.8 mm, vias 0 -> 3
- net VBUS: track 0.00 -> 102.2 mm
- net I2C_SMBALERT: track 0.00 -> 97.1 mm, vias 0 -> 2
- net NRST_RADIO_MCU: track 0.00 -> 91.8 mm, vias 0 -> 2
- net BAT-: track 0.00 -> 87.0 mm, vias 0 -> 29
- net SPI_SCK: track 0.00 -> 74.2 mm, vias 0 -> 4
- net SPI_MOSI: track 0.00 -> 64.7 mm, vias 0 -> 3
- net SPI_MISO: track 0.00 -> 63.3 mm, vias 0 -> 3
- net RADIO_DIO5: track 0.00 -> 58.6 mm, vias 0 -> 2
- net RADIO_TX: track 0.00 -> 53.3 mm, vias 0 -> 3
- net RADIO_NSS: track 0.00 -> 33.5 mm, vias 0 -> 3
- net RADIO_RST: track 0.00 -> 32.9 mm, vias 0 -> 3
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- added copper zone on F.Cu, net 3.3V
- added copper zone on B.Cu, net BAT-
Other:
- board size 55.9 x 92.7 mm -> 55.9 x 98.2 mm
- board text added: "+sw"
- board text added: "100nF"
- board text added: "10kΩ"
- board text added: "1k5Ω"
- board text added: "1kΩ"
- board text added: "1uF"
- board text added: "20pF"
- board text added: "4k7Ω"
- board text added: "68Ω"
- board text added: "ALERT"
- board text added: "MAIN_TX"
- board text added: "PCONN"
- board text added: "RADIO_TX"
- board text removed: "++"
- board text removed: "PERIPHERAL"
- board text removed: "SMBALERT"
- board text removed: "SW_BAT"

Commit message: Update production
Parts:
- added G***: LOGO, powiloc-custom:pollex-logo, B.Cu at (142.7, 64.5)
- added REF**: OSHW-Logo2_9.8x8mm_SilkScreen, Symbol:OSHW-Logo2_9.8x8mm_SilkScreen, B.Cu at (163.6, 97.0)
Routing:
- net VBUS: track 102.2 -> 104.9 mm
